Commit message: Add Lidar on Go2

File: robots/go2_description/xacro/go2_generated.urdf (robot description, URDF)
Before this commit: robot go2, 19 links, 18 joints
Links:
- added link hokuyo_frame, mass 0.270; collision box size=0.058 0.058 0.087; visual mesh filename=package://hector_sensors_description/meshes/hokuyo_utm30lx/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
Joints:
- added joint hokuyo_joint: type fixed, parent trunk, child hokuyo_frame, origin xyz=0.0 0.0 0.096 rpy=0 0 0
