Commit message: mod parent link velodyne joint

File: robots/go2_description/xacro/go2_velodyne_description.urdf (robot description, URDF)
Before this commit: robot go2, 21 links, 20 joints
Joints:
- joint velodyne_base_mount_joint: origin xyz=0 0 0.11 rpy=0 0 0 -> xyz=0 0 0.096 rpy=0 0 0; parent base -> trunk

Commit message: mod go2 velodyne

File: robots/go2_description/xacro/go2_velodyne_description.urdf (robot description, URDF)
Before this commit: robot go2, 21 links, 20 joints
Links:
- link velodyne_base_link: mass 0.83 -> 0.01
Joints:
- joint velodyne_base_mount_joint: origin xyz=0 0 0.096 rpy=0 0 0 -> xyz=0.2 0 0.08 rpy=0 0 0
